Commit message: Update USD and URDF with new per-component export

File: robot_description/urdf/Floyd_URDF.urdf (robot description, URDF)
Before this commit: robot BDX_Robot, 12 links, 11 joints
Links:
- added link Back_Base, mass 0.101249; collision mesh filename=package://Floyd_URDF_description/meshes/Floyd_URDF/Back_Bas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 scale=0.01 0.01 0.01; visual mesh filename=package://Floyd_URDF_description/meshes/Floyd_URDF/Back_Bas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 scale=1 1 1
- added link Battery, mass 1.273; collision mesh filename=package://Floyd_URDF_description/meshes/Floyd_URDF/Battery_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 scale=0.01 0.01 0.01; visual mesh filename=package://Floyd_URDF_description/meshes/Floyd_URDF/Battery.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 scale=1 1 1
- added link Battery_Mount, mass 0.046707; collision mesh filename=package://Floyd_URDF_description/meshes/Floyd_URDF/Battery_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 scale=0.01 0.01 0.01; visual mesh filename=package://Floyd_URDF_description/meshes/Floyd_URDF/Battery_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 scale=1 1 1
- added link BellyBase, mass 0.098302; collision mesh filename=package://Floyd_URDF_description/meshes/Floyd_URDF/BellyBas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 scale=0.01 0.01 0.01; visual mesh filename=package://Floyd_URDF_description/meshes/Floyd_URDF/BellyBas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 scale=1 1 1
- added link FootBaseLeft, mass 0.12934; collision mesh filename=package://Floyd_URDF_description/meshes/Floyd_URDF/FootBase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 scale=0.01 0.01 0.01; visual mesh filename=package://Floyd_URDF_description/meshes/Floyd_URDF/FootBase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 scale=1 1 1
- added link FootCoverLeft, mass 0.025806; collision mesh filename=package://Floyd_URDF_description/meshes/Floyd_URDF/FootCove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 scale=0.01 0.01 0.01; visual mesh filename=package://Floyd_URDF_description/meshes/Floyd_URDF/FootCove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 scale=1 1 1
- added link FrontBase, mass 0.138068; collision mesh filename=package://Floyd_URDF_description/meshes/Floyd_URDF/FrontBas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 scale=0.01 0.01 0.01; visual mesh filename=package://Floyd_URDF_description/meshes/Floyd_URDF/FrontBas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 scale=1 1 1
- added link FrontPanel, mass 0.124478; collision mesh filename=package://Floyd_URDF_description/meshes/Floyd_URDF/FrontPan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 scale=0.01 0.01 0.01; visual mesh filename=package://Floyd_URDF_description/meshes/Floyd_URDF/FrontPan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 scale=1 1 1
- added link LowerLegLeft, mass 0.203942; collision mesh filename=package://Floyd_URDF_description/meshes/Floyd_URDF/LowerLeg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 scale=0.01 0.01 0.01; visual mesh filename=package://Floyd_URDF_description/meshes/Floyd_URDF/LowerLeg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 scale=1 1 1
- added link LowerLegRight, mass 0.203942; collision mesh filename=package://Floyd_URDF_description/meshes/Floyd_URDF/LowerLeg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 scale=0.01 0.01 0.01; visual mesh filename=package://Floyd_URDF_description/meshes/Floyd_URDF/LowerLeg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 scale=1 1 1
- added link LowerPanel, mass 0.017805; collision mesh filename=package://Floyd_URDF_description/meshes/Floyd_URDF/LowerPan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 scale=0.01 0.01 0.01
- added link RS02, mass 0.412; collision mesh filename=package://Floyd_URDF_description/meshes/Floyd_URDF/RS02_col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 scale=0.01 0.01 0.01; visual mesh filename=package://Floyd_URDF_description/meshes/Floyd_URDF/RS02.dae scale=1 1 1
- added link RS03_LeftHipRoll, mass 0.88; collision mesh filename=package://Floyd_URDF_description/meshes/Floyd_URDF/RS03_Lef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 scale=0.01 0.01 0.01; visual mesh filename=package://Floyd_URDF_description/meshes/Floyd_URDF/RS03_Lef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 scale=1 1 1
- added link RS03_LeftKneePitch, mass 0.88; collision mesh filename=package://Floyd_URDF_description/meshes/Floyd_URDF/RS03_Lef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 scale=0.01 0.01 0.01; visual mesh filename=package://Floyd_URDF_description/meshes/Floyd_URDF/RS03_Lef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 scale=1 1 1
- added link RS03_RightHipPitch, mass 0.88; collision mesh filename=package://Floyd_URDF_description/meshes/Floyd_URDF/RS03_Rig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 scale=0.01 0.01 0.01; visual mesh filename=package://Floyd_URDF_description/meshes/Floyd_URDF/RS03_Rig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 scale=1 1 1
- added link RS03_RightHipRoll, mass 0.88; collision mesh filename=package://Floyd_URDF_description/meshes/Floyd_URDF/RS03_Rig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 scale=0.01 0.01 0.01; visual mesh filename=package://Floyd_URDF_description/meshes/Floyd_URDF/RS03_Rig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 scale=1 1 1
- added link Tail_Base, mass 0.094793; collision mesh filename=package://Floyd_URDF_description/meshes/Floyd_URDF/Tail_Bas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 scale=0.01 0.01 0.01; visual mesh filename=package://Floyd_URDF_description/meshes/Floyd_URDF/Tail_Bas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 scale=1 1 1
- added link ThighMountFemaleLeft, mass 0.235725; collision mesh filename=package://Floyd_URDF_description/meshes/Floyd_URDF/ThighMou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 scale=0.01 0.01 0.01; visual mesh filename=package://Floyd_URDF_description/meshes/Floyd_URDF/ThighMou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 scale=1 1 1
- added link ThighMountFemaleRight, mass 0.235725; collision mesh filename=package://Floyd_URDF_description/meshes/Floyd_URDF/ThighMou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 scale=0.01 0.01 0.01; visual mesh filename=package://Floyd_URDF_description/meshes/Floyd_URDF/ThighMou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 scale=1 1 1
- added link ThighMountMaleLeft, mass 0.196896; collision mesh filename=package://Floyd_URDF_description/meshes/Floyd_URDF/ThighMou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 scale=0.01 0.01 0.01; visual mesh filename=package://Floyd_URDF_description/meshes/Floyd_URDF/ThighMou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 scale=1 1 1
- added link ThighMountMaleRight, mass 0.196896; collision mesh filename=package://Floyd_URDF_description/meshes/Floyd_URDF/ThighMou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 scale=0.01 0.01 0.01; visual mesh filename=package://Floyd_URDF_description/meshes/Floyd_URDF/ThighMou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 scale=1 1 1
- added link TopBase, mass 0.086052; collision mesh filename=package://Floyd_URDF_description/meshes/Floyd_URDF/TopBase_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 scale=0.01 0.01 0.01; visual mesh filename=package://Floyd_URDF_description/meshes/Floyd_URDF/TopBase.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 scale=1 1 1
- added link TopLeftPanel, mass 0.017563; collision mesh filename=package://Floyd_URDF_description/meshes/Floyd_URDF/TopLeftP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 scale=0.01 0.01 0.01; visual mesh filename=package://Floyd_URDF_description/meshes/Floyd_URDF/TopLeftP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 scale=1 1 1
- added link TopRightPanel, mass 0.017563; collision mesh filename=package://Floyd_URDF_description/meshes/Floyd_URDF/TopRight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 scale=0.01 0.01 0.01; visual mesh filename=package://Floyd_URDF_description/meshes/Floyd_URDF/TopRight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 scale=1 1 1
- link FootBaseRight: mass 0.129 -> 0.12934
- link FootCoverRight: mass 0.026 -> 0.025807
- link FootPadLeft: mass 0.210 -> 0.79727
- link FootPadRight: mass 0.055 -> 0.797489
- link HipRollMountLeft: mass 0.089 -> 0.099119
- link HipRollMountRight: mass 0.089 -> 0.099119
- link RS02_LeftAnklePitch: mass 0.544 -> 0.412
- link RS02_RightAnklePitch: mass 0.544 -> 0.412
- link RS03_LeftHipPitch: mass 2.170 -> 0.88
- link RS03_RightKneePitch: mass 2.170 -> 0.88
- link base_link: mass 4.537 -> 0.394155
Joints:
- added joint Rigid_17: type fixed, parent ThighMountFemaleLeft, child ThighMountMaleLeft, origin xyz=0.000000 0.000000 -0.000000 rpy=-0.000000 0.000000 0.000000
- added joint Rigid_21: type fixed, parent FootBaseLeft, child FootCoverLeft, origin xyz=-0.118071 -0.137704 0.226786 rpy=0.000000 0.000000 0.000000
- added joint Rigid_23: type fixed, parent LowerLegLeft, child RS02_LeftAnklePitch, origin xyz=-0.001500 -0.140028 -0.000013 rpy=-1.570796 -0.261799 -1.570796
- added joint Rigid_25: type fixed, parent FootBaseLeft, child FootPadLeft, origin xyz=-0.118071 -0.138154 0.226886 rpy=0.000000 0.000000 -0.000000
- added joint Rigid_28: type fixed, parent LowerLegRight, child RS02_RightAnklePitch, origin xyz=-0.001500 -0.140028 0.000013 rpy=1.570796 0.261799 -1.570796
- added joint Rigid_29: type fixed, parent ThighMountFemaleRight, child ThighMountMaleRight, origin xyz=0.000000 0.000000 0.000000 rpy=0.000000 -0.000000 -0.000000
- added joint Rigid_47: type fixed, parent base_link, child RS02, origin xyz=0.013750 0.200264 0.011850 rpy=-1.570796 -0.000000 -1.570796
- added joint Rigid_48: type fixed, parent base_link, child BellyBase, origin xyz=-0.000393 0.133156 0.057146 rpy=-1.570796 -0.000000 0.000000
- added joint Rigid_49: type fixed, parent base_link, child FrontBase, origin xyz=-0.000393 0.133156 0.056746 rpy=-1.570796 -0.000000 0.000000
- added joint Rigid_50: type fixed, parent base_link, child Back_Base, origin xyz=0.000000 0.000000 0.000150 rpy=-0.000000 0.000000 -0.000000
- added joint Rigid_51: type fixed, parent Back_Base, child Tail_Base, origin xyz=0.000000 0.000000 0.000000 rpy=0.000000 0.000000 0.000000
- added joint Rigid_52: type fixed, parent Back_Base, child Battery_Mount, origin xyz=0.000000 0.000000 0.000000 rpy=0.000000 0.000000 0.000000
- added joint Rigid_53: type fixed, parent Battery_Mount, child Battery, origin xyz=0.000050 0.005043 0.000000 rpy=0.000000 0.000000 0.000000
- added joint Rigid_54: type fixed, parent base_link, child RS03_LeftHipRoll, origin xyz=0.050050 0.102099 -0.090118 rpy=0.000001 0.000000 -1.570796
- added joint Rigid_55: type fixed, parent base_link, child RS03_RightHipRoll, origin xyz=-0.049950 0.102099 -0.090118 rpy=-0.000001 0.000000 1.570796
- added joint Rigid_56: type fixed, parent TopBase, child TopRightPanel, origin xyz=0.000443 -0.000104 -0.000000 rpy=-3.141593 -0.000000 3.141593
- added joint Rigid_57: type fixed, parent TopBase, child TopLeftPanel, origin xyz=0.000443 -0.000104 -0.000000 rpy=0.000000 -0.000000 -0.000000
- added joint Rigid_58: type fixed, parent BellyBase, child FrontPanel, origin xyz=0.000443 -0.000104 -0.000000 rpy=0.000000 0.000000 0.000000
- added joint Rigid_59: type fixed, parent RS03_LeftHipPitch, child ThighMountFemaleLeft, origin xyz=-0.058592 0.000000 0.071250 rpy=0.000000 1.570796 0.000000
- added joint Rigid_61: type fixed, parent RS03_RightHipPitch, child ThighMountFemaleRight, origin xyz=0.058592 0.000000 0.071250 rpy=-0.000000 1.570796 0.000000
- added joint Rigid_63: type fixed, parent BellyBase, child LowerPanel, origin xyz=-0.000000 0.000000 0.000000 rpy=0.000000 0.000000 0.000000
- added joint Rigid_64: type fixed, parent ThighMountFemaleLeft, child RS03_LeftKneePitch, origin xyz=0.127850 -0.111000 0.058592 rpy=-0.000000 -1.570796 0.000000
- added joint Rigid_65: type fixed, parent ThighMountFemaleRight, child RS03_RightKneePitch, origin xyz=0.127850 -0.111000 -0.058593 rpy=-0.000000 1.570796 0.000000
- added joint Rigid_66: type fixed, parent FrontBase, child TopBase, origin xyz=-0.000000 -0.000000 -0.000200 rpy=0.000000 -0.000000 0.000000
- joint LeftAnklePitch: axis 1.000000 -0.000000 -0.000000 -> 1.000000 0.000000 -0.000000; child FootPadLeft -> FootBaseLeft; limit lower=-0.785000 upper=1.221730 effort=17.0 velocity=43.0 -> lower= upper= effort=17.0 velocity=43.0; origin xyz=0.135254 0.036254 0.002500 rpy=0.436332 -1.570796 0.000000 -> xyz=0.000000 0.000000 0.004000 rpy=0.436332 -1.570796 0.000000
- joint LeftHipPitch: limit lower=-0.698132 upper=1.047198 effort=60.0 velocity=20.0 -> lower= upper= effort=60.0 velocity=20.0; origin xyz=0.071250 -0.000000 0.012092 rpy=-1.570796 0.698132 1.570796 -> xyz=0.071250 -0.000000 0.012093 rpy=-1.570796 0.698132 1.570796
- joint LeftHipRoll: limit lower=-0.349066 upper=0.261799 effort=60.0 velocity=20.0 -> lower= upper= effort=60.0 velocity=20.0; origin xyz=0.098165 0.045368 0.036300 rpy=-0.000000 -1.570795 -1.570796 -> xyz=0.000000 -0.000000 0.056600 rpy=3.141593 0.000000 1.570796; parent base_link -> RS03_LeftHipRoll
- joint LeftKneePitch: axis 0.000000 0.000000 -1.000000 -> -1.000000 0.000000 0.000000; child RS02_LeftAnklePitch -> LowerLegLeft; limit lower=-1.308997 upper=0.959931 effort=60.0 velocity=20.0 -> lower= upper= effort=60.0 velocity=20.0; origin xyz=0.000000 -0.111000 -0.000000 rpy=3.141593 -0.000000 -0.261799 -> xyz=-0.000000 -0.000000 0.056600 rpy=-1.047198 1.570796 0.000000; parent RS03_LeftHipPitch -> RS03_LeftKneePitch
- joint RightAnklePitch: axis -1.000000 0.000000 0.000000 -> -1.000000 -0.000000 -0.000000; limit lower=-0.785000 upper=1.221730 effort=17.0 velocity=43.0 -> lower= upper= effort=17.0 velocity=43.0; origin xyz=0.135254 0.036254 -0.002500 rpy=-0.436332 1.570796 0.000000 -> xyz=0.000000 -0.000000 -0.004000 rpy=-0.436332 1.570796 0.000000
- joint RightHipPitch: axis -0.000000 -0.000000 1.000000 -> 0.000000 0.000000 -1.000000; child RS03_RightKneePitch -> RS03_RightHipPitch; limit lower=-1.047198 upper=0.698132 effort=60.0 velocity=20.0 -> lower= upper= effort=60.0 velocity=20.0; origin xyz=0.071250 -0.000000 -0.012092 rpy=1.570796 -0.698132 1.570796 -> xyz=0.071250 -0.000000 -0.012092 rpy=1.570796 0.698132 -1.570796
- joint RightHipRoll: limit lower=-0.349066 upper=0.261799 effort=60.0 velocity=20.0 -> lower= upper= effort=60.0 velocity=20.0; origin xyz=0.098165 0.045368 -0.063700 rpy=-3.141593 1.570795 1.570796 -> xyz=0.000000 -0.000000 0.056600 rpy=-0.000000 0.000000 1.570796; parent base_link -> RS03_RightHipRoll
- joint RightKneePitch: axis 0.000000 -0.000000 -1.000000 -> 1.000000 -0.000000 0.000000; child RS02_RightAnklePitch -> LowerLegRight; limit lower=-1.308997 upper=0.959931 effort=60.0 velocity=20.0 -> lower= upper= effort=60.0 velocity=20.0; origin xyz=0.000000 -0.111000 0.000000 rpy=-3.141593 -0.000000 -0.261799 -> xyz=0.000000 0.000000 -0.056600 rpy=1.047198 -1.570796 0.000000
- joint Rigid_45: origin xyz=-0.118071 -0.137704 -0.226786 rpy=0 0 0 -> xyz=-0.118071 -0.137704 -0.226786 rpy=-0.000000 -0.000000 -0.000000
- joint Rigid_46: origin xyz=-0.118071 -0.138154 -0.226886 rpy=0 0 0 -> xyz=-0.118071 -0.138154 -0.226886 rpy=-0.000000 0.000000 0.000000
- joint world_to_base: origin xyz=0 0 0.35 rpy=0 1.5708 0 -> xyz=0 0 0.07 rpy=1.5708 0 0
