Commit message: Fix PD gains, obs scales, teleop script, ankle penalty during yaw turns

File: robot_description/urdf/Floyd_URDF_original.urdf (robot description, URDF)
Before this commit: robot BDX_Robot, 36 links, 35 joints
Links:
- link base_link: geometry collision mesh filename=package://Floyd_URDF_description/meshes/Floyd_URDF/base_lin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 scale=0.01 0.01 0.01; visual mesh filename=package://Floyd_URDF_description/meshes/Floyd_URDF/base_lin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 scale=1 1 1

File: robot_description/usd/Floyd_URDF_description/urdf/Floyd_URDF.urdf (robot description, URDF)
Before this commit: robot BDX_Robot, 36 links, 35 joints
Links:
- link base_link: geometry collision mesh filename=package://Floyd_URDF_description/meshes/Floyd_URDF/base_lin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 scale=0.01 0.01 0.01; visual mesh filename=package://Floyd_URDF_description/meshes/Floyd_URDF/base_lin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 scale=1 1 1
Joints:
- joint LeftAnklePitch: limit lower= upper= effort=17.0 velocity=43.0 -> lower=-0.5236 upper=1.2217 effort=17.0 velocity=43.0
- joint LeftHipPitch: limit lower= upper= effort=60.0 velocity=20.0 -> lower=-1.0472 upper=0.6981 effort=60.0 velocity=20.0
- joint LeftHipRoll: limit lower= upper= effort=60.0 velocity=20.0 -> lower=-0.3491 upper=0.3491 effort=60.0 velocity=20.0
- joint LeftKneePitch: limit lower= upper= effort=60.0 velocity=20.0 -> lower=-0.1745 upper=1.0472 effort=60.0 velocity=20.0
- joint RightAnklePitch: limit lower= upper= effort=17.0 velocity=43.0 -> lower=-0.5236 upper=1.2217 effort=17.0 velocity=43.0
- joint RightHipPitch: limit lower= upper= effort=60.0 velocity=20.0 -> lower=-0.6981 upper=1.0472 effort=60.0 velocity=20.0
- joint RightHipRoll: limit lower= upper= effort=60.0 velocity=20.0 -> lower=-0.3491 upper=0.3491 effort=60.0 velocity=20.0
- joint RightKneePitch: limit lower= upper= effort=60.0 velocity=20.0 -> lower=-0.1745 upper=1.0472 effort=60.0 velocity=20.0
- joint world_to_base: origin xyz=0 0 0.07 rpy=1.5708 0 0 -> xyz=0 0 0.07 rpy=1.5708 0 1.5708
